Commit message: feat(experiments): structure multi-experiment workspace and add joint limits experiment

File: output/virgo_gimbal_compiled.urdf (robot description, URDF)
Before this commit: robot virgo_gimbal_payload, 17 links, 16 joints
Joints:
- joint j_gimbal_motor_1: limit (none) -> lower=-1.5708 upper=0.7854 effort=1.2 velocity=6.28319; type continuous -> revolute
- joint j_gimbal_motor_2: limit (none) -> lower=-0.7854 upper=0.7854 effort=1.2 velocity=6.28319; type continuous -> revolute
- joint j_gimbal_motor_3: limit (none) -> lower=-2.79253 upper=2.79253 effort=1.5 velocity=6.28319; type continuous -> revolute
