Commit message: refactor(exp03): map internal nomenclature and preserve baseline artifacts

File: experiments/03_cad_coordinate_alignment/xacro/virgo_gimbal.xacro (robot description, xacro)
@@ -5,8 +5,8 @@
   <xacro:macro name="virgo_gimbal">
     <!-- =================================================================== -->
-    <!-- 10 Kinematic Links                                                  -->
+    <!-- 10 Kinematic Links (Internal Standard Nomenclature)                 -->
     <!-- =================================================================== -->
-    <!-- 1. ISP Box Mount Link (Kinematic Root) -->
-    <link name="isp_box_link">
+    <!-- 1. ISP Box Mount Link (Kinematic Root Base) -->
+    <link name="gimbal_mnt_link">
       <visual>
         <origin xyz="0 0 0" rpy="0 0 0" />
@@ -16,6 +16,6 @@
       </visual>
     </link>
-    <!-- 2. Suspension Frame Link -->
-    <link name="suspend_link">
+    <!-- 2. Suspension Dampening Plate Link -->
+    <link name="gimbal_susp_link">
       <visual>
         <origin xyz="0 0 0" rpy="0 0 0" />
@@ -25,6 +25,6 @@
       </visual>
     </link>
-    <!-- 3. Roll Axis Gimbal Link -->
-    <link name="roll_link">
+    <!-- 3. Roll Axis Motor Link (Motor 3) -->
+    <link name="gimbal_motor_3_link">
       <visual>
         <origin xyz="0 0 0" rpy="0 0 0" />
@@ -34,6 +34,6 @@
       </visual>
     </link>
-    <!-- 4. Yaw Axis Gimbal Link -->
-    <link name="yaw_link">
+    <!-- 4. Yaw Axis Motor Link (Motor 2) -->
+    <link name="gimbal_motor_2_link">
       <visual>
         <origin xyz="0 0 0" rpy="0 0 0" />
@@ -43,6 +43,6 @@
       </visual>
     </link>
-    <!-- 5. Pitch Axis Gimbal Link -->
-    <link name="pitch_link">
+    <!-- 5. Pitch Axis Motor Link (Motor 1) -->
+    <link name="gimbal_motor_1_link">
       <visual>
         <origin xyz="0 0 0" rpy="0 0 0" />
@@ -53,5 +53,5 @@
     </link>
     <!-- 6. Sensor Payload Bracket Link -->
-    <link name="payload_link">
+    <link name="gimbal_payload_link">
       <visual>
         <origin xyz="0 0 0" rpy="0 0 0" />
@@ -61,6 +61,6 @@
       </visual>
     </link>
-    <!-- 7. IMU Sensor Link -->
-    <link name="imu_link">
+    <!-- 7. IMU Sensor Link Frame -->
+    <link name="imu_1_frame">
       <visual>
         <origin xyz="0 0 0" rpy="0 0 0" />
@@ -71,5 +71,5 @@
     </link>
     <!-- 8. Narrow Camera Sensor Link -->
-    <link name="narrow_cam_link">
+    <link name="cam_narrow_link">
       <visual>
         <origin xyz="0 0 0" rpy="0 0 0" />
@@ -80,5 +80,5 @@
     </link>
     <!-- 9. Telephoto Camera Sensor Link -->
-    <link name="tele_cam_link">
+    <link name="cam_tele_link">
       <visual>
         <origin xyz="0 0 0" rpy="0 0 0" />
@@ -89,5 +89,5 @@
     </link>
     <!-- 10. Wide Camera Sensor Link -->
-    <link name="wide_cam_link">
+    <link name="cam_wide_link">
       <visual>
         <origin xyz="0 0 0" rpy="0 0 0" />
@@ -98,66 +98,66 @@
     </link>
     <!-- =================================================================== -->
-    <!-- 9 Kinematic Transformation Joints                                   -->
-    <!-- Topology: ISP BOX -> Suspend -> Roll -> Yaw -> Pitch -> Payload     -->
-    <!--           Payload -> (IMU / Narrow / Tele / Wide)                   -->
+    <!-- 9 Kinematic Transformation Joints (Internal Standard Nomenclature)  -->
+    <!-- Topology: Mount -> Suspension -> Motor 3 (Roll) -> Motor 2 (Yaw) -> -->
+    <!--           Motor 1 (Pitch) -> Payload -> (IMU / Narrow / Tele / Wide)-->
     <!-- =================================================================== -->
-    <!-- Joint 1: ISP Box to Suspend (Fixed) -->
-    <joint name="isp_box_to_suspend" type="fixed">
-      <parent link="isp_box_link" />
-      <child link="suspend_link" />
+    <!-- Joint 1: Mount Base to Suspension (Fixed) -->
+    <joint name="gimbal_mnt_to_susp_joint" type="fixed">
+      <parent link="gimbal_mnt_link" />
+      <child link="gimbal_susp_link" />
       <origin xyz="${isp_box_to_suspend_xyz}" rpy="${isp_box_to_suspend_rpy}" />
     </joint>
-    <!-- Joint 2: Suspend to Roll Axis (Revolute) -->
-    <joint name="suspend_to_roll" type="revolute">
-      <parent link="suspend_link" />
-      <child link="roll_link" />
+    <!-- Joint 2: Suspension to Motor 3 / Roll Axis (Revolute) -->
+    <joint name="gimbal_susp_to_motor3_joint" type="revolute">
+      <parent link="gimbal_susp_link" />
+      <child link="gimbal_motor_3_link" />
       <origin xyz="${suspend_to_roll_xyz}" rpy="${suspend_to_roll_rpy}" />
       <axis xyz="1 0 0" />
       <limit lower="-0.785398" upper="0.785398" effort="10.0" velocity="1.0" />
     </joint>
-    <!-- Joint 3: Roll to Yaw Axis (Revolute) -->
-    <joint name="roll_to_yaw" type="revolute">
-      <parent link="roll_link" />
-      <child link="yaw_link" />
+    <!-- Joint 3: Motor 3 to Motor 2 / Yaw Axis (Revolute) -->
+    <joint name="gimbal_motor3_to_motor2_joint" type="revolute">
+      <parent link="gimbal_motor_3_link" />
+      <child link="gimbal_motor_2_link" />
       <origin xyz="${roll_to_yaw_xyz}" rpy="${roll_to_yaw_rpy}" />
       <axis xyz="0 0 1" />
       <limit lower="-2.79253" upper="2.79253" effort="10.0" velocity="1.0" />
     </joint>
-    <!-- Joint 4: Yaw to Pitch Axis (Revolute) -->
-    <joint name="yaw_to_pitch" type="revolute">
-      <parent link="yaw_link" />
-      <child link="pitch_link" />
+    <!-- Joint 4: Motor 2 to Motor 1 / Pitch Axis (Revolute) -->
+    <joint name="gimbal_motor2_to_motor1_joint" type="revolute">
+      <parent link="gimbal_motor_2_link" />
+      <child link="gimbal_motor_1_link" />
       <origin xyz="${yaw_to_pitch_xyz}" rpy="${yaw_to_pitch_rpy}" />
       <axis xyz="0 1 0" />
       <limit lower="-1.5708" upper="0.785398" effort="10.0" velocity="1.0" />
     </joint>
-    <!-- Joint 5: Pitch to Payload Bracket (Fixed) -->
-    <joint name="pitch_to_payload" type="fixed">
-      <parent link="pitch_link" />
-      <child link="payload_link" />
+    <!-- Joint 5: Motor 1 to Payload Bracket (Fixed) -->
+    <joint name="gimbal_motor1_to_payload_joint" type="fixed">
+      <parent link="gimbal_motor_1_link" />
+      <child link="gimbal_payload_link" />
       <origin xyz="${pitch_to_payload_xyz}" rpy="${pitch_to_payload_rpy}" />
     </joint>
     <!-- Joint 6: Payload to IMU (Fixed) -->
-    <joint name="payload_to_imu" type="fixed">
-      <parent link="payload_link" />
-      <child link="imu_link" />
+    <joint name="gimbal_payload_to_imu_joint" type="fixed">
+      <parent link="gimbal_payload_link" />
+      <child link="imu_1_frame" />
       <origin xyz="${payload_to_imu_xyz}" rpy="${payload_to_imu_rpy}" />
     </joint>
     <!-- Joint 7: Payload to Narrow Camera (Fixed) -->
-    <joint name="payload_to_narrow" type="fixed">
-      <parent link="payload_link" />
-      <child link="narrow_cam_link" />
+    <joint name="gimbal_payload_to_narrow_joint" type="fixed">
+      <parent link="gimbal_payload_link" />
+      <child link="cam_narrow_link" />
       <origin xyz="${payload_to_narrow_xyz}" rpy="${payload_to_narrow_rpy}" />
     </joint>
     <!-- Joint 8: Payload to Tele Camera (Fixed) -->
-    <joint name="payload_to_tele" type="fixed">
-      <parent link="payload_link" />
-      <child link="tele_cam_link" />
+    <joint name="gimbal_payload_to_tele_joint" type="fixed">
+      <parent link="gimbal_payload_link" />
+      <child link="cam_tele_link" />
       <origin xyz="${payload_to_tele_xyz}" rpy="${payload_to_tele_rpy}" />
     </joint>
     <!-- Joint 9: Payload to Wide Camera (Fixed) -->
-    <joint name="payload_to_wide" type="fixed">
-      <parent link="payload_link" />
-      <child link="wide_cam_link" />
+    <joint name="gimbal_payload_to_wide_joint" type="fixed">
+      <parent link="gimbal_payload_link" />
+      <child link="cam_wide_link" />
       <origin xyz="${payload_to_wide_xyz}" rpy="${payload_to_wide_rpy}" />
     </joint>

File: output/03_cad_coordinate_alignment/virgo_gimbal_compiled.urdf (robot description, URDF)
Before this commit: robot virgo_gimbal_exp03, 10 links, 9 joints
Links:
- removed link imu_link
- removed link isp_box_link
- removed link narrow_cam_link
- removed link payload_link
- removed link pitch_link
- removed link roll_link
- removed link suspend_link
- removed link tele_cam_link
- removed link wide_cam_link
- removed link yaw_link
- added link cam_narrow_link; visual cylinder length=0.025 radius=0.012
- added link cam_tele_link; visual cylinder length=0.035 radius=0.015
- added link cam_wide_link; visual cylinder length=0.020 radius=0.010
- added link gimbal_mnt_link; visual box size=0.08 0.08 0.04
- added link gimbal_motor_1_link; visual cylinder length=0.04 radius=0.02
- added link gimbal_motor_2_link; visual cylinder length=0.04 radius=0.02
- added link gimbal_motor_3_link; visual cylinder length=0.04 radius=0.02
- added link gimbal_payload_link; visual box size=0.10 0.06 0.05
- added link gimbal_susp_link; visual box size=0.07 0.07 0.02
- added link imu_1_frame; visual box size=0.015 0.015 0.008
Joints:
- removed joint isp_box_to_suspend
- removed joint payload_to_imu
- removed joint payload_to_narrow
- removed joint payload_to_tele
- removed joint payload_to_wide
- removed joint pitch_to_payload
- removed joint roll_to_yaw
- removed joint suspend_to_roll
- removed joint yaw_to_pitch
- added joint gimbal_mnt_to_susp_joint: type fixed, parent gimbal_mnt_link, child gimbal_susp_link, origin xyz=0.064306 -0.000001 0.021546 rpy=0.0 0.0 0.0
- added joint gimbal_motor1_to_payload_joint: type fixed, parent gimbal_motor_1_link, child gimbal_payload_link, origin xyz=-0.000069 -0.000666 0.060957 rpy=-1.570796 0.0 -2.783801
- added joint gimbal_motor2_to_motor1_joint: type revolute, parent gimbal_motor_2_link, child gimbal_motor_1_link, origin xyz=0.0 0.054600 0.078100 rpy=1.570796 1.570796 0.0, axis 0 1 0, limit lower=-1.5708 upper=0.785398 effort=10.0 velocity=1.0
- added joint gimbal_motor3_to_motor2_joint: type revolute, parent gimbal_motor_3_link, child gimbal_motor_2_link, origin xyz=-0.039807 0.0 0.034129 rpy=0.0 0.750491 0.0, axis 0 0 1, limit lower=-2.79253 upper=2.79253 effort=10.0 velocity=1.0
- added joint gimbal_payload_to_imu_joint: type fixed, parent gimbal_payload_link, child imu_1_frame, origin xyz=-0.018398 0.022833 0.023084 rpy=3.141593 1.570796 0.0
- added joint gimbal_payload_to_narrow_joint: type fixed, parent gimbal_payload_link, child cam_narrow_link, origin xyz=-0.025633 0.016500 -0.013660 rpy=-1.570796 0.0 -1.570796
- added joint gimbal_payload_to_tele_joint: type fixed, parent gimbal_payload_link, child cam_tele_link, origin xyz=-0.025633 -0.016500 -0.013660 rpy=-1.570796 0.0 -1.570796
- added joint gimbal_payload_to_wide_joint: type fixed, parent gimbal_payload_link, child cam_wide_link, origin xyz=0.017012 -0.000740 0.014340 rpy=-1.570796 0.0 -1.570796
- added joint gimbal_susp_to_motor3_joint: type revolute, parent gimbal_susp_link, child gimbal_motor_3_link, origin xyz=-0.070790 0.0 0.029217 rpy=0.0 1.178098 0.0, axis 1 0 0, limit lower=-0.785398 upper=0.785398 effort=10.0 velocity=1.0

File: output/03_cad_coordinate_alignment/virgo_gimbal_raw_compiled.urdf (robot description, URDF)
Before this commit: robot virgo_gimbal_exp03, 10 links, 9 joints
Joints:
- joint isp_box_to_suspend: origin xyz=0.0 0.0 0.0 rpy=0.0 0.0 0.0 -> xyz=0.064306 -0.000001 0.021546 rpy=0.0 0.0 0.0
- joint payload_to_imu: origin xyz=0.0 0.0 0.0 rpy=0.0 0.0 0.0 -> xyz=-0.018398 0.022833 0.023084 rpy=3.141593 1.570796 0.0
- joint payload_to_narrow: origin xyz=0.0 0.0 0.0 rpy=0.0 0.0 0.0 -> xyz=-0.025633 0.016500 -0.013660 rpy=-1.570796 0.0 -1.570796
- joint payload_to_tele: origin xyz=0.0 0.0 0.0 rpy=0.0 0.0 0.0 -> xyz=-0.025633 -0.016500 -0.013660 rpy=-1.570796 0.0 -1.570796
- joint payload_to_wide: origin xyz=0.0 0.0 0.0 rpy=0.0 0.0 0.0 -> xyz=0.017012 -0.000740 0.014340 rpy=-1.570796 0.0 -1.570796
- joint pitch_to_payload: origin xyz=0.0 0.0 0.0 rpy=0.0 0.0 0.0 -> xyz=-0.000069 -0.000666 0.060957 rpy=-1.570796 0.0 -2.783801
- joint roll_to_yaw: origin xyz=0.0 0.0 0.0 rpy=0.0 0.0 0.0 -> xyz=-0.039807 0.0 0.034129 rpy=0.0 0.750491 0.0
- joint suspend_to_roll: origin xyz=0.0 0.0 0.0 rpy=0.0 0.0 0.0 -> xyz=-0.070790 0.0 0.029217 rpy=0.0 1.178098 0.0
- joint yaw_to_pitch: origin xyz=0.0 0.0 0.0 rpy=0.0 0.0 0.0 -> xyz=0.0 0.054600 0.078100 rpy=1.570796 1.570796 0.0
