Commit message: feat(exp03): apply ER_260820 exact cad transforms and generate kinematic artifacts

File: experiments/03_cad_coordinate_alignment/xacro/virgo_cad_transforms.xacro (robot description, xacro)
@@ -5,36 +5,36 @@
     Vendor CAD Transformation Specifications (ER_260820 Baseline)
     ===========================================================================
-    This file contains pre-reserved transformation properties derived from
-    vendor CAD Datum Coordinate Systems (CAD_Model_ER_260820).
+    This file contains exact transformation properties derived from vendor CAD
+    Datum Coordinate Systems (CAD_Model_ER_260820).
     Units:
       - Translational (xyz): Meters [m] (converted from millimeters)
-      - Rotational (rpy): Radians [rad] (converted from degrees)
+      - Rotational (rpy): Radians [rad] (converted from Euler angles / matrix)
   -->
   <!-- 1. ISP Box -> Suspend Transform -->
-  <xacro:property name="isp_box_to_suspend_xyz" value="0.0 0.0 0.0" />
+  <xacro:property name="isp_box_to_suspend_xyz" value="0.064306 -0.000001 0.021546" />
   <xacro:property name="isp_box_to_suspend_rpy" value="0.0 0.0 0.0" />
   <!-- 2. Suspend -> Roll Transform -->
-  <xacro:property name="suspend_to_roll_xyz" value="0.0 0.0 0.0" />
-  <xacro:property name="suspend_to_roll_rpy" value="0.0 0.0 0.0" />
+  <xacro:property name="suspend_to_roll_xyz" value="-0.070790 0.0 0.029217" />
+  <xacro:property name="suspend_to_roll_rpy" value="0.0 1.178098 0.0" />
   <!-- 3. Roll -> Yaw Transform -->
-  <xacro:property name="roll_to_yaw_xyz" value="0.0 0.0 0.0" />
-  <xacro:property name="roll_to_yaw_rpy" value="0.0 0.0 0.0" />
+  <xacro:property name="roll_to_yaw_xyz" value="-0.039807 0.0 0.034129" />
+  <xacro:property name="roll_to_yaw_rpy" value="0.0 0.750491 0.0" />
   <!-- 4. Yaw -> Pitch Transform -->
-  <xacro:property name="yaw_to_pitch_xyz" value="0.0 0.0 0.0" />
-  <xacro:property name="yaw_to_pitch_rpy" value="0.0 0.0 0.0" />
+  <xacro:property name="yaw_to_pitch_xyz" value="0.0 0.054600 0.078100" />
+  <xacro:property name="yaw_to_pitch_rpy" value="1.570796 1.570796 0.0" />
   <!-- 5. Pitch -> Payload Transform -->
-  <xacro:property name="pitch_to_payload_xyz" value="0.0 0.0 0.0" />
-  <xacro:property name="pitch_to_payload_rpy" value="0.0 0.0 0.0" />
+  <xacro:property name="pitch_to_payload_xyz" value="-0.000069 -0.000666 0.060957" />
+  <xacro:property name="pitch_to_payload_rpy" value="-1.570796 0.0 -2.783801" />
   <!-- 6. Payload -> IMU Transform -->
-  <xacro:property name="payload_to_imu_xyz" value="0.0 0.0 0.0" />
-  <xacro:property name="payload_to_imu_rpy" value="0.0 0.0 0.0" />
+  <xacro:property name="payload_to_imu_xyz" value="-0.018398 0.022833 0.023084" />
+  <xacro:property name="payload_to_imu_rpy" value="3.141593 1.570796 0.0" />
   <!-- 7. Payload -> Narrow Camera Transform -->
-  <xacro:property name="payload_to_narrow_xyz" value="0.0 0.0 0.0" />
-  <xacro:property name="payload_to_narrow_rpy" value="0.0 0.0 0.0" />
+  <xacro:property name="payload_to_narrow_xyz" value="-0.025633 0.016500 -0.013660" />
+  <xacro:property name="payload_to_narrow_rpy" value="-1.570796 0.0 -1.570796" />
   <!-- 8. Payload -> Tele Camera Transform -->
-  <xacro:property name="payload_to_tele_xyz" value="0.0 0.0 0.0" />
-  <xacro:property name="payload_to_tele_rpy" value="0.0 0.0 0.0" />
+  <xacro:property name="payload_to_tele_xyz" value="-0.025633 -0.016500 -0.013660" />
+  <xacro:property name="payload_to_tele_rpy" value="-1.570796 0.0 -1.570796" />
   <!-- 9. Payload -> Wide Camera Transform -->
-  <xacro:property name="payload_to_wide_xyz" value="0.0 0.0 0.0" />
-  <xacro:property name="payload_to_wide_rpy" value="0.0 0.0 0.0" />
+  <xacro:property name="payload_to_wide_xyz" value="0.017012 -0.000740 0.014340" />
+  <xacro:property name="payload_to_wide_rpy" value="-1.570796 0.0 -1.570796" />
 </robot>

Commit message: feat(exp03): append standard cv frames (*_cv_frame) to camera links

File: experiments/03_cad_coordinate_alignment/xacro/virgo_cad_transforms.xacro (robot description, xacro)
@@ -38,3 +38,6 @@
   <xacro:property name="payload_to_wide_xyz" value="0.017012 -0.000740 0.014340" />
   <xacro:property name="payload_to_wide_rpy" value="-1.570796 0.0 -1.570796" />
+  <!-- 10. Camera Link -> OpenCV Visual Frame Transform -->
+  <xacro:property name="cam_link_to_cv_xyz" value="0.0 0.0 0.0" />
+  <xacro:property name="cam_link_to_cv_rpy" value="-1.570796 0.0 -1.570796" />
 </robot>

File: experiments/03_cad_coordinate_alignment/xacro/virgo_gimbal.xacro (robot description, xacro)
@@ -5,5 +5,5 @@
   <xacro:macro name="virgo_gimbal">
     <!-- =================================================================== -->
-    <!-- 10 Kinematic Links (Internal Standard Nomenclature)                 -->
+    <!-- 13 Kinematic Links (Internal Standard Nomenclature & OpenCV Frames) -->
     <!-- =================================================================== -->
     <!-- 1. ISP Box Mount Link (Kinematic Root Base) -->
@@ -97,8 +97,15 @@
       </visual>
     </link>
+    <!-- 11. Narrow Camera OpenCV Visual Frame Link -->
+    <link name="cam_narrow_cv_frame" />
+    <!-- 12. Telephoto Camera OpenCV Visual Frame Link -->
+    <link name="cam_tele_cv_frame" />
+    <!-- 13. Wide Camera OpenCV Visual Frame Link -->
+    <link name="cam_wide_cv_frame" />
     <!-- =================================================================== -->
-    <!-- 9 Kinematic Transformation Joints (Internal Standard Nomenclature)  -->
+    <!-- 12 Kinematic Transformation Joints (Internal Standard Nomenclature) -->
     <!-- Topology: Mount -> Suspension -> Motor 3 (Roll) -> Motor 2 (Yaw) -> -->
     <!--           Motor 1 (Pitch) -> Payload -> (IMU / Narrow / Tele / Wide)-->
+    <!--           -> (Narrow_CV / Tele_CV / Wide_CV)                        -->
     <!-- =================================================================== -->
     <!-- Joint 1: Mount Base to Suspension (Fixed) -->
@@ -162,4 +169,22 @@
       <origin xyz="${payload_to_wide_xyz}" rpy="${payload_to_wide_rpy}" />
     </joint>
+    <!-- Joint 10: Narrow Camera Link to OpenCV Visual Frame (Fixed) -->
+    <joint name="cam_narrow_cv_j" type="fixed">
+      <parent link="cam_narrow_link" />
+      <child link="cam_narrow_cv_frame" />
+      <origin xyz="${cam_link_to_cv_xyz}" rpy="${cam_link_to_cv_rpy}" />
+    </joint>
+    <!-- Joint 11: Tele Camera Link to OpenCV Visual Frame (Fixed) -->
+    <joint name="cam_tele_cv_j" type="fixed">
+      <parent link="cam_tele_link" />
+      <child link="cam_tele_cv_frame" />
+      <origin xyz="${cam_link_to_cv_xyz}" rpy="${cam_link_to_cv_rpy}" />
+    </joint>
+    <!-- Joint 12: Wide Camera Link to OpenCV Visual Frame (Fixed) -->
+    <joint name="cam_wide_cv_j" type="fixed">
+      <parent link="cam_wide_link" />
+      <child link="cam_wide_cv_frame" />
+      <origin xyz="${cam_link_to_cv_xyz}" rpy="${cam_link_to_cv_rpy}" />
+    </joint>
   </xacro:macro>
 </robot>

File: output/03_cad_coordinate_alignment/virgo_gimbal_compiled.urdf (robot description, URDF)
Before this commit: robot virgo_gimbal_exp03, 10 links, 9 joints
Links:
- added link cam_narrow_cv_frame
- added link cam_tele_cv_frame
- added link cam_wide_cv_frame
Joints:
- added joint cam_narrow_cv_j: type fixed, parent cam_narrow_link, child cam_narrow_cv_frame, origin xyz=0.0 0.0 0.0 rpy=-1.570796 0.0 -1.570796
- added joint cam_tele_cv_j: type fixed, parent cam_tele_link, child cam_tele_cv_frame, origin xyz=0.0 0.0 0.0 rpy=-1.570796 0.0 -1.570796
- added joint cam_wide_cv_j: type fixed, parent cam_wide_link, child cam_wide_cv_frame, origin xyz=0.0 0.0 0.0 rpy=-1.570796 0.0 -1.570796

Commit message: fix(exp03): align camera body frames with rep-103 zero-rotation and isolate optical cv transform

File: experiments/03_cad_coordinate_alignment/xacro/virgo_cad_transforms.xacro (robot description, xacro)
@@ -29,13 +29,13 @@
   <xacro:property name="payload_to_imu_xyz" value="-0.018398 0.022833 0.023084" />
   <xacro:property name="payload_to_imu_rpy" value="3.141593 1.570796 0.0" />
-  <!-- 7. Payload -> Narrow Camera Transform -->
+  <!-- 7. Payload -> Narrow Camera Transform (REP-103 Body Frame Alignment) -->
   <xacro:property name="payload_to_narrow_xyz" value="-0.025633 0.016500 -0.013660" />
-  <xacro:property name="payload_to_narrow_rpy" value="-1.570796 0.0 -1.570796" />
-  <!-- 8. Payload -> Tele Camera Transform -->
+  <xacro:property name="payload_to_narrow_rpy" value="0.0 0.0 0.0" />
+  <!-- 8. Payload -> Tele Camera Transform (REP-103 Body Frame Alignment) -->
   <xacro:property name="payload_to_tele_xyz" value="-0.025633 -0.016500 -0.013660" />
-  <xacro:property name="payload_to_tele_rpy" value="-1.570796 0.0 -1.570796" />
-  <!-- 9. Payload -> Wide Camera Transform -->
+  <xacro:property name="payload_to_tele_rpy" value="0.0 0.0 0.0" />
+  <!-- 9. Payload -> Wide Camera Transform (REP-103 Body Frame Alignment) -->
   <xacro:property name="payload_to_wide_xyz" value="0.017012 -0.000740 0.014340" />
-  <xacro:property name="payload_to_wide_rpy" value="-1.570796 0.0 -1.570796" />
+  <xacro:property name="payload_to_wide_rpy" value="0.0 0.0 0.0" />
   <!-- 10. Camera Link -> OpenCV Visual Frame Transform -->
   <xacro:property name="cam_link_to_cv_xyz" value="0.0 0.0 0.0" />

File: output/03_cad_coordinate_alignment/virgo_gimbal_compiled.urdf (robot description, URDF)
Before this commit: robot virgo_gimbal_exp03, 13 links, 12 joints
Joints:
- joint gimbal_payload_to_narrow_joint: origin xyz=-0.025633 0.016500 -0.013660 rpy=-1.570796 0.0 -1.570796 -> xyz=-0.025633 0.016500 -0.013660 rpy=0.0 0.0 0.0
- joint gimbal_payload_to_tele_joint: origin xyz=-0.025633 -0.016500 -0.013660 rpy=-1.570796 0.0 -1.570796 -> xyz=-0.025633 -0.016500 -0.013660 rpy=0.0 0.0 0.0
- joint gimbal_payload_to_wide_joint: origin xyz=0.017012 -0.000740 0.014340 rpy=-1.570796 0.0 -1.570796 -> xyz=0.017012 -0.000740 0.014340 rpy=0.0 0.0 0.0
